Commit message: add hardware interface tag to joints

File: urdf/youbot_arm/arm.transmission.xacro (robot description, xacro)
@@ -13,5 +13,7 @@
         <mechanicalReduction>1</mechanicalReduction>
       </actuator>
-			<joint name="${name}_joint_1"/>
+			<joint name="${name}_joint_1">
+        <hardwareInterface>EffortJointInterface</hardwareInterface>
+      </joint>
 		</transmission>
 		<transmission name="${name}_trans_2">
@@ -21,5 +23,7 @@
         <mechanicalReduction>1</mechanicalReduction>
       </actuator>
-			<joint name="${name}_joint_2"/>
+			<joint name="${name}_joint_2">
+        <hardwareInterface>EffortJointInterface</hardwareInterface>
+      </joint>
 		</transmission>
 		<transmission name="${name}_trans_3">
@@ -29,5 +33,7 @@
         <mechanicalReduction>1</mechanicalReduction>
       </actuator>
-			<joint name="${name}_joint_3"/>
+			<joint name="${name}_joint_3">
+        <hardwareInterface>EffortJointInterface</hardwareInterface>
+      </joint>
 		</transmission>
 		<transmission name="${name}_trans_4">
@@ -37,5 +43,7 @@
         <mechanicalReduction>1</mechanicalReduction>
       </actuator>
-			<joint name="${name}_joint_4"/>
+			<joint name="${name}_joint_4">
+        <hardwareInterface>EffortJointInterface</hardwareInterface>
+      </joint>
 		</transmission>
 		<transmission name="${name}_trans_5">
@@ -45,5 +53,7 @@
         <mechanicalReduction>1</mechanicalReduction>
       </actuator>
-			<joint name="${name}_joint_5"/>
+			<joint name="${name}_joint_5">
+        <hardwareInterface>EffortJointInterface</hardwareInterface>
+      </joint>
 		</transmission>
 	</xacro:macro>

File: urdf/youbot_base/base.transmission.xacro (robot description, xacro)
@@ -15,5 +15,7 @@
         <mechanicalReduction>${wheel_mechanical_reduction}</mechanicalReduction>
       </actuator>
-			<joint name="wheel_joint_fl" />
+			<joint name="wheel_joint_fl">
+        <hardwareInterface>VelocityJointInterface</hardwareInterface>
+      </joint>
 		</transmission>
 		<transmission name="caster_trans_fl">
@@ -23,5 +25,7 @@
         <mechanicalReduction>${caster_mechanical_reduction}</mechanicalReduction>
       </actuator>
-      <joint name="caster_joint_fl" />
+      <joint name="caster_joint_fl">
+        <hardwareInterface>VelocityJointInterface</hardwareInterface>
+      </joint>
     </transmission>
 	  <!-- front right wheel -->
@@ -32,5 +36,7 @@
         <mechanicalReduction>${wheel_mechanical_reduction}</mechanicalReduction>
       </actuator>
-		  <joint name="wheel_joint_fr" />
+		  <joint name="wheel_joint_fr">
+        <hardwareInterface>VelocityJointInterface</hardwareInterface>
+      </joint>
 	  </transmission>
 	  <transmission name="caster_trans_fr">
@@ -40,5 +46,7 @@
         <mechanicalReduction>${caster_mechanical_reduction}</mechanicalReduction>
       </actuator>
-    	<joint name="caster_joint_fr" />
+      <joint name="caster_joint_fr">
+        <hardwareInterface>VelocityJointInterface</hardwareInterface>
+      </joint>
     </transmission>
 	  <!-- back left wheel -->
@@ -49,5 +57,7 @@
         <mechanicalReduction>${wheel_mechanical_reduction}</mechanicalReduction>
       </actuator>
-	    <joint name="wheel_joint_bl" />
+	    <joint name="wheel_joint_bl">
+        <hardwareInterface>VelocityJointInterface</hardwareInterface>
+      </joint>
 	  </transmission>
 	  <transmission name="caster_trans_bl">
@@ -57,5 +67,7 @@
         <mechanicalReduction>${caster_mechanical_reduction}</mechanicalReduction>
       </actuator>
-    	<joint name="caster_joint_bl" />
+      <joint name="caster_joint_bl">
+        <hardwareInterface>VelocityJointInterface</hardwareInterface>
+      </joint>
     </transmission>
 	  <!-- back right wheel -->
@@ -66,5 +78,7 @@
         <mechanicalReduction>${wheel_mechanical_reduction}</mechanicalReduction>
       </actuator>
-		  <joint name="wheel_joint_br" />
+		  <joint name="wheel_joint_br">
+        <hardwareInterface>VelocityJointInterface</hardwareInterface>
+      </joint>
 	  </transmission>
 	  <transmission name="caster_trans_br">
@@ -74,5 +88,7 @@
         <mechanicalReduction>${caster_mechanical_reduction}</mechanicalReduction>
       </actuator>
-    	<joint name="caster_joint_br" />
+      <joint name="caster_joint_br">
+        <hardwareInterface>VelocityJointInterface</hardwareInterface>
+      </joint>
     </transmission>
   </xacro:macro>

File: urdf/youbot_gripper/gripper.transmission.xacro (robot description, xacro)
@@ -11,5 +11,7 @@
         <mechanicalReduction>1</mechanicalReduction>
       </actuator>
-			<joint name="${name}_finger_joint_l"/>
+			<joint name="${name}_finger_joint_l">
+        <hardwareInterface>EffortJointInterface</hardwareInterface>
+      </joint>
 		</transmission>
 		<transmission name="${name}_finger_r_trans">
@@ -19,5 +21,7 @@
         <mechanicalReduction>1</mechanicalReduction>
       </actuator>
-			<joint name="${name}_finger_joint_r"/>
+			<joint name="${name}_finger_joint_r">
+        <hardwareInterface>EffortJointInterface</hardwareInterface>
+      </joint>
 		</transmission>
 	</xacro:macro>

Commit message: added HardwareInterface in joints for newer Gazebo versions, corrected indentation

File: urdf/youbot_arm/arm.transmission.xacro (robot description, xacro)
@@ -8,42 +8,52 @@
 	<xacro:macro name="youbot_arm_transmission" params="name">
 		<transmission name="${name}_trans_1">
-      <type>transmission_interface/SimpleTransmission</type>
+			<type>transmission_interface/SimpleTransmission</type>
 			<actuator name="${name}_motor_1">
-        <hardwareInterface>EffortJointInterface</hardwareInterface>
-        <mechanicalReduction>1</mechanicalReduction>
-      </actuator>
-			<joint name="${name}_joint_1"/>
+				<hardwareInterface>EffortJointInterface</hardwareInterface>
+				<mechanicalReduction>1</mechanicalReduction>
+			</actuator>
+			<joint name="${name}_joint_1">
+				<hardwareInterface>EffortJointInterface</hardwareInterface>
+			</joint>
 		</transmission>
 		<transmission name="${name}_trans_2">
-      <type>transmission_interface/SimpleTransmission</type>
+			<type>transmission_interface/SimpleTransmission</type>
 			<actuator name="${name}_motor_2">
-        <hardwareInterface>EffortJointInterface</hardwareInterface>
-        <mechanicalReduction>1</mechanicalReduction>
-      </actuator>
-			<joint name="${name}_joint_2"/>
+				<hardwareInterface>EffortJointInterface</hardwareInterface>
+				<mechanicalReduction>1</mechanicalReduction>
+			</actuator>
+			<joint name="${name}_joint_2">
+				<hardwareInterface>EffortJointInterface</hardwareInterface>
+			</joint>
 		</transmission>
 		<transmission name="${name}_trans_3">
-      <type>transmission_interface/SimpleTransmission</type>
+			<type>transmission_interface/SimpleTransmission</type>
 			<actuator name="${name}_motor_3">
-        <hardwareInterface>EffortJointInterface</hardwareInterface>
-        <mechanicalReduction>1</mechanicalReduction>
-      </actuator>
-			<joint name="${name}_joint_3"/>
+				<hardwareInterface>EffortJointInterface</hardwareInterface>
+				<mechanicalReduction>1</mechanicalReduction>
+			</actuator>
+			<joint name="${name}_joint_3">
+				<hardwareInterface>EffortJointInterface</hardwareInterface>
+			</joint>
 		</transmission>
 		<transmission name="${name}_trans_4">
-      <type>transmission_interface/SimpleTransmission</type>
+			<type>transmission_interface/SimpleTransmission</type>
 			<actuator name="${name}_motor_4">
-        <hardwareInterface>EffortJointInterface</hardwareInterface>
-        <mechanicalReduction>1</mechanicalReduction>
-      </actuator>
-			<joint name="${name}_joint_4"/>
+				<hardwareInterface>EffortJointInterface</hardwareInterface>
+				<mechanicalReduction>1</mechanicalReduction>
+			</actuator>
+			<joint name="${name}_joint_4">
+				<hardwareInterface>EffortJointInterface</hardwareInterface>
+			</joint>
 		</transmission>
 		<transmission name="${name}_trans_5">
-      <type>transmission_interface/SimpleTransmission</type>
+			<type>transmission_interface/SimpleTransmission</type>
 			<actuator name="${name}_motor_5">
-        <hardwareInterface>EffortJointInterface</hardwareInterface>
-        <mechanicalReduction>1</mechanicalReduction>
-      </actuator>
-			<joint name="${name}_joint_5"/>
+				<hardwareInterface>EffortJointInterface</hardwareInterface>
+				<mechanicalReduction>1</mechanicalReduction>
+			</actuator>
+			<joint name="${name}_joint_5">
+				<hardwareInterface>EffortJointInterface</hardwareInterface>
+			</joint>
 		</transmission>
 	</xacro:macro>

File: urdf/youbot_base/base.transmission.xacro (robot description, xacro)
@@ -6,74 +6,90 @@
 	<property name="wheel_mechanical_reduction" value="${624/35 * 80/18}" />
 	<property name="caster_mechanical_reduction" value="${624/35 * 80/18}" />
-  <property name="" value="0.360" />
+	<property name="" value="0.360" />
 	<xacro:macro name="youbot_base_transmission">
-	<!-- front left wheel -->
+		<!-- front left wheel -->
 		<transmission name="wheel_trans_fl">
-      <type>transmission_interface/SimpleTransmission</type>
+			<type>transmission_interface/SimpleTransmission</type>
 			<actuator name="wheel_motor_fl">
-        <hardwareInterface>VelocityJointInterface</hardwareInterface>
-        <mechanicalReduction>${wheel_mechanical_reduction}</mechanicalReduction>
-      </actuator>
-			<joint name="wheel_joint_fl" />
+				<hardwareInterface>VelocityJointInterface</hardwareInterface>
+				<mechanicalReduction>${wheel_mechanical_reduction}</mechanicalReduction>
+			</actuator>
+			<joint name="wheel_joint_fl">
+				<hardwareInterface>VelocityJointInterface</hardwareInterface>
+			</joint>
 		</transmission>
 		<transmission name="caster_trans_fl">
-      <type>transmission_interface/SimpleTransmission</type>
-   	  <actuator name="caster_motor_fl">
-        <hardwareInterface>VelocityJointInterface</hardwareInterface>
-        <mechanicalReduction>${caster_mechanical_reduction}</mechanicalReduction>
-      </actuator>
-      <joint name="caster_joint_fl" />
-    </transmission>
-	  <!-- front right wheel -->
-	  <transmission name="wheel_trans_fr">
-      <type>transmission_interface/SimpleTransmission</type>
-		  <actuator name="wheel_motor_fr">
-        <hardwareInterface>VelocityJointInterface</hardwareInterface>
-        <mechanicalReduction>${wheel_mechanical_reduction}</mechanicalReduction>
-      </actuator>
-		  <joint name="wheel_joint_fr" />
-	  </transmission>
-	  <transmission name="caster_trans_fr">
-      <type>transmission_interface/SimpleTransmission</type>
-      <actuator name="caster_motor_fr" >
-        <hardwareInterface>VelocityJointInterface</hardwareInterface>
-        <mechanicalReduction>${caster_mechanical_reduction}</mechanicalReduction>
-      </actuator>
-    	<joint name="caster_joint_fr" />
-    </transmission>
-	  <!-- back left wheel -->
-	  <transmission name="wheel_trans_bl">
-      <type>transmission_interface/SimpleTransmission</type>
-	    <actuator name="wheel_motor_bl" >
-        <hardwareInterface>VelocityJointInterface</hardwareInterface>
-        <mechanicalReduction>${wheel_mechanical_reduction}</mechanicalReduction>
-      </actuator>
-	    <joint name="wheel_joint_bl" />
-	  </transmission>
-	  <transmission name="caster_trans_bl">
-      <type>transmission_interface/SimpleTransmission</type>
-      <actuator name="caster_motor_bl" >
-        <hardwareInterface>VelocityJointInterface</hardwareInterface>
-        <mechanicalReduction>${caster_mechanical_reduction}</mechanicalReduction>
-      </actuator>
-    	<joint name="caster_joint_bl" />
-    </transmission>
-	  <!-- back right wheel -->
-	  <transmission name="wheel_trans_br">
-      <type>transmission_interface/SimpleTransmission</type>
-	    <actuator name="wheel_motor_br" >
-        <hardwareInterface>VelocityJointInterface</hardwareInterface>
-        <mechanicalReduction>${wheel_mechanical_reduction}</mechanicalReduction>
-      </actuator>
-		  <joint name="wheel_joint_br" />
-	  </transmission>
-	  <transmission name="caster_trans_br">
-      <type>transmission_interface/SimpleTransmission</type>
-      <actuator name="caster_motor_br" >
-        <hardwareInterface>VelocityJointInterface</hardwareInterface>
-        <mechanicalReduction>${caster_mechanical_reduction}</mechanicalReduction>
-      </actuator>
-    	<joint name="caster_joint_br" />
-    </transmission>
-  </xacro:macro>
+			<type>transmission_interface/SimpleTransmission</type>
+			<actuator name="caster_motor_fl">
+				<hardwareInterface>VelocityJointInterface</hardwareInterface>
+				<mechanicalReduction>${caster_mechanical_reduction}</mechanicalReduction>
+			</actuator>
+			<joint name="caster_joint_fl">
+				<hardwareInterface>VelocityJointInterface</hardwareInterface>
+			</joint>
+		</transmission>
+		<!-- front right wheel -->
+		<transmission name="wheel_trans_fr">
+			<type>transmission_interface/SimpleTransmission</type>
+			<actuator name="wheel_motor_fr">
+				<hardwareInterface>VelocityJointInterface</hardwareInterface>
+				<mechanicalReduction>${wheel_mechanical_reduction}</mechanicalReduction>
+			</actuator>
+			<joint name="wheel_joint_fr">
+				<hardwareInterface>VelocityJointInterface</hardwareInterface>
+			</joint>
+		</transmission>
+		<transmission name="caster_trans_fr">
+			<type>transmission_interface/SimpleTransmission</type>
+			<actuator name="caster_motor_fr" >
+				<hardwareInterface>VelocityJointInterface</hardwareInterface>
+				<mechanicalReduction>${caster_mechanical_reduction}</mechanicalReduction>
+			</actuator>
+			<joint name="caster_joint_fr">
+				<hardwareInterface>VelocityJointInterface</hardwareInterface>
+			</joint>
+		</transmission>
+		<!-- back left wheel -->
+		<transmission name="wheel_trans_bl">
+			<type>transmission_interface/SimpleTransmission</type>
+			<actuator name="wheel_motor_bl" >
+				<hardwareInterface>VelocityJointInterface</hardwareInterface>
+				<mechanicalReduction>${wheel_mechanical_reduction}</mechanicalReduction>
+			</actuator>
+			<joint name="wheel_joint_bl">
+				<hardwareInterface>VelocityJointInterface</hardwareInterface>
+			</joint>
+		</transmission>
+		<transmission name="caster_trans_bl">
+			<type>transmission_interface/SimpleTransmission</type>
+			<actuator name="caster_motor_bl" >
+				<hardwareInterface>VelocityJointInterface</hardwareInterface>
+				<mechanicalReduction>${caster_mechanical_reduction}</mechanicalReduction>
+			</actuator>
+			<joint name="caster_joint_bl">
+				<hardwareInterface>VelocityJointInterface</hardwareInterface>
+			</joint>
+		</transmission>
+		<!-- back right wheel -->
+		<transmission name="wheel_trans_br">
+			<type>transmission_interface/SimpleTransmission</type>
+			<actuator name="wheel_motor_br" >
+				<hardwareInterface>VelocityJointInterface</hardwareInterface>
+				<mechanicalReduction>${wheel_mechanical_reduction}</mechanicalReduction>
+			</actuator>
+			<joint name="wheel_joint_br">
+				<hardwareInterface>VelocityJointInterface</hardwareInterface>
+			</joint>
+		</transmission>
+		<transmission name="caster_trans_br">
+			<type>transmission_interface/SimpleTransmission</type>
+			<actuator name="caster_motor_br" >
+				<hardwareInterface>VelocityJointInterface</hardwareInterface>
+				<mechanicalReduction>${caster_mechanical_reduction}</mechanicalReduction>
+			</actuator>
+			<joint name="caster_joint_br">
+				<hardwareInterface>VelocityJointInterface</hardwareInterface>
+			</joint>
+		</transmission>
+	</xacro:macro>
 </robot>

File: urdf/youbot_gripper/gripper.transmission.xacro (robot description, xacro)
@@ -6,18 +6,22 @@
 	<xacro:macro name="youbot_gripper_transmission" params="name">
 		<transmission name="${name}_finger_l_trans">
-      <type>transmission_interface/SimpleTransmission</type>
+			<type>transmission_interface/SimpleTransmission</type>
 			<actuator name="${name}_finger_l_motor">
-        <hardwareInterface>EffortJointInterface</hardwareInterface>
-        <mechanicalReduction>1</mechanicalReduction>
-      </actuator>
-			<joint name="${name}_finger_joint_l"/>
+				<hardwareInterface>EffortJointInterface</hardwareInterface>
+				<mechanicalReduction>1</mechanicalReduction>
+			</actuator>
+			<joint name="${name}_finger_joint_l">
+				<hardwareInterface>EffortJointInterface</hardwareInterface>
+			</joint>
 		</transmission>
 		<transmission name="${name}_finger_r_trans">
-      <type>transmission_interface/SimpleTransmission</type>
+			<type>transmission_interface/SimpleTransmission</type>
 			<actuator name="${name}_finger_r_motor">
-        <hardwareInterface>EffortJointInterface</hardwareInterface>
-        <mechanicalReduction>1</mechanicalReduction>
-      </actuator>
-			<joint name="${name}_finger_joint_r"/>
+				<hardwareInterface>EffortJointInterface</hardwareInterface>
+				<mechanicalReduction>1</mechanicalReduction>
+			</actuator>
+			<joint name="${name}_finger_joint_r">
+				<hardwareInterface>EffortJointInterface</hardwareInterface>
+			</joint>
 		</transmission>
 	</xacro:macro>
