Commit message: Updated xml namespace tags

File: robots/youbot_arm_only.urdf.xacro (robot description, xacro)
@@ -1,8 +1,4 @@
 <?xml version="1.0"?>
-<robot xmlns:sensor="http://playerstage.sourceforge.net/gazebo/xmlschema/#sensor"
-       xmlns:controller="http://playerstage.sourceforge.net/gazebo/xmlschema/#controller"
-       xmlns:interface="http://playerstage.sourceforge.net/gazebo/xmlschema/#interface"
-       xmlns:xacro="http://playerstage.sourceforge.net/gazebo/xmlschema/#interface"
-       name="youbot" >
+<robot xmlns:xacro="http://ros.org/wiki/xacro" name="youbot" >
   <!-- The following included files set up definitions of parts of the robot body -->
   <!-- misc common stuff? -->

File: urdf/materials.urdf.xacro (robot description, xacro)
@@ -1,4 +1,4 @@
 <?xml version="1.0"?>
-<robot>
+<robot xmlns:xacro="http://www.ros.org/wiki/xacro">
   <material name="Orange">
     <color rgba="1.0 0.4 0.0 1.0"/>

File: urdf/youbot_arm/arm.gazebo.xacro (robot description, xacro)
@@ -1,7 +1,4 @@
 <?xml version="1.0"?>
-<robot xmlns:sensor="http://playerstage.sourceforge.net/gazebo/xmlschema/#sensor"
-       xmlns:controller="http://playerstage.sourceforge.net/gazebo/xmlschema/#controller"
-       xmlns:interface="http://playerstage.sourceforge.net/gazebo/xmlschema/#interface"
-       xmlns:xacro="http://ros.org/wiki/xacro">
+<robot xmlns:xacro="http://ros.org/wiki/xacro">
 	<xacro:macro name="youbot_arm_gazebo" params="name">
 		<gazebo reference="${name}_link_0">

File: urdf/youbot_arm/arm.transmission.xacro (robot description, xacro)
@@ -1,7 +1,4 @@
 <?xml version="1.0"?>
-<robot xmlns:sensor="http://playerstage.sourceforge.net/gazebo/xmlschema/#sensor"
-       xmlns:controller="http://playerstage.sourceforge.net/gazebo/xmlschema/#controller"
-       xmlns:interface="http://playerstage.sourceforge.net/gazebo/xmlschema/#interface"
-       xmlns:xacro="http://ros.org/wiki/xacro">
+<robot xmlns:xacro="http://ros.org/wiki/xacro">
 	<!-- reduction ratio doesn't affect the model-->
 	<!-- reduction ratio must not to be 0-->
@@ -14,5 +11,5 @@
 			</actuator>
 			<joint name="${name}_joint_1">
-				<hardwareInterface>EffortJointInterface</hardwareInterface>
+				<hardwareInterface>hardware_interface/EffortJointInterface</hardwareInterface>
 			</joint>
 		</transmission>
@@ -24,5 +21,5 @@
 			</actuator>
 			<joint name="${name}_joint_2">
-				<hardwareInterface>EffortJointInterface</hardwareInterface>
+				<hardwareInterface>hardware_interface/EffortJointInterface</hardwareInterface>
 			</joint>
 		</transmission>
@@ -34,5 +31,5 @@
 			</actuator>
 			<joint name="${name}_joint_3">
-				<hardwareInterface>EffortJointInterface</hardwareInterface>
+				<hardwareInterface>hardware_interface/EffortJointInterface</hardwareInterface>
 			</joint>
 		</transmission>
@@ -44,5 +41,5 @@
 			</actuator>
 			<joint name="${name}_joint_4">
-				<hardwareInterface>EffortJointInterface</hardwareInterface>
+				<hardwareInterface>hardware_interface/EffortJointInterface</hardwareInterface>
 			</joint>
 		</transmission>
@@ -54,5 +51,5 @@
 			</actuator>
 			<joint name="${name}_joint_5">
-				<hardwareInterface>EffortJointInterface</hardwareInterface>
+				<hardwareInterface>hardware_interface/EffortJointInterface</hardwareInterface>
 			</joint>
 		</transmission>

File: urdf/youbot_arm/arm.urdf.xacro (robot description, xacro)
@@ -1,7 +1,4 @@
 <?xml version="1.0"?>
-<robot  xmlns:sensor="http://playerstage.sourceforge.net/gazebo/xmlschema/#sensor"
-        xmlns:controller="http://playerstage.sourceforge.net/gazebo/xmlschema/#controller"
-        xmlns:interface="http://playerstage.sourceforge.net/gazebo/xmlschema/#interface"
-        xmlns:xacro="http://ros.org/wiki/xacro">
+<robot  xmlns:xacro="http://ros.org/wiki/xacro">
 	<xacro:include filename="$(find youbot_description)/urdf/youbot_arm/arm.gazebo.xacro" />
 	<xacro:include filename="$(find youbot_description)/urdf/youbot_arm/arm.transmission.xacro" />
@@ -10,5 +7,5 @@
 		<!-- joint between base_link and arm_0_link -->
 		<joint name="${name}_joint_0" type="fixed" >
-			<insert_block name="origin" />
+			<xacro:insert_block name="origin" />
 			<parent link="${parent}" />
 			<child link="${name}_link_0" />
@@ -211,4 +208,11 @@
 			</collision>
 		</link>
+        <joint name="${name}_joint_ee" type="fixed">
+          <parent link="${name}_link_5"/>
+          <child link="${name}_link_ee"/>
+          <origin xyz="0 0 0.045" rpy="0 0 0"/>
+        </joint>
+        <link name="${name}_link_ee">
+        </link>
 		<!-- extensions -->
 		<xacro:youbot_arm_gazebo name="${name}" />

File: urdf/youbot_arm/limits.urdf.xacro (robot description, xacro)
@@ -1,31 +1,31 @@
 <?xml version="1.0"?>
-<robot xmlns:xacro="http://ros.org/wiki/xacro">>
+<robot xmlns:xacro="http://ros.org/wiki/xacro">
 	<!-- common properties -->
-	<property name="M_PI" value="3.1415926535897931" />
-        <property name="threshold" value="0.01" />
+	<xacro:property name="M_PI" value="3.1415926535897931" />
+        <xacro:property name="threshold" value="0.01" />
 	<!-- arm limits positions (deg) -->
-	<property name="joint_1_limit" value="${M_PI * (169 + 169) / 180}" />
-	<property name="joint_2_limit" value="${M_PI * (90 + 65) / 180}" />
-	<property name="joint_3_limit" value="${M_PI * (146 + 151) / 180}" />
-	<property name="joint_4_limit" value="${M_PI * (102.5 + 102.5) / 180}" />
-	<property name="joint_5_limit" value="${M_PI * (167.5 + 167.5) / 180}" />
-        <property name="joint_1_limit_soft" value="${M_PI * (169 + 169) / 180 - threshold}" />
-	<property name="joint_2_limit_soft" value="${M_PI * (90 + 65) / 180 - threshold}" />
-	<property name="joint_3_limit_soft" value="${M_PI * (146 + 151) / 180 - threshold}" />
-	<property name="joint_4_limit_soft" value="${M_PI * (102.5 + 102.5) / 180 - threshold}" />
-	<property name="joint_5_limit_soft" value="${M_PI * (167.5 + 167.5) / 180 - threshold}" />
+	<xacro:property name="joint_1_limit" value="${M_PI * (169 + 169) / 180}" />
+	<xacro:property name="joint_2_limit" value="${M_PI * (90 + 65) / 180}" />
+	<xacro:property name="joint_3_limit" value="${M_PI * (146 + 151) / 180}" />
+	<xacro:property name="joint_4_limit" value="${M_PI * (102.5 + 102.5) / 180}" />
+	<xacro:property name="joint_5_limit" value="${M_PI * (167.5 + 167.5) / 180}" />
+        <xacro:property name="joint_1_limit_soft" value="${M_PI * (169 + 169) / 180 - threshold}" />
+	<xacro:property name="joint_2_limit_soft" value="${M_PI * (90 + 65) / 180 - threshold}" />
+	<xacro:property name="joint_3_limit_soft" value="${M_PI * (146 + 151) / 180 - threshold}" />
+	<xacro:property name="joint_4_limit_soft" value="${M_PI * (102.5 + 102.5) / 180 - threshold}" />
+	<xacro:property name="joint_5_limit_soft" value="${M_PI * (167.5 + 167.5) / 180 - threshold}" />
 	<!-- dynamic properties : mass (kg) Alu data sheet -->
-	<property name="link_0_mass" value="0.845" />
-	<property name="link_1_mass" value="2.412" />
-	<property name="link_2_mass" value="1.155" />
-	<property name="link_3_mass" value="0.934" />
-	<property name="link_4_mass" value="0.877" />
-	<property name="link_5_mass" value="0.251" />
-	<!--<property name="link_0_mass" value="0.845" />
-	<property name="link_1_mass" value="0.1" />
-	<property name="link_2_mass" value="0.1" />
-	<property name="link_3_mass" value="0.1" />
-	<property name="link_4_mass" value="0.1" />
-	<property name="link_5_mass" value="0.1" />-->
+	<xacro:property name="link_0_mass" value="0.845" />
+	<xacro:property name="link_1_mass" value="2.412" />
+	<xacro:property name="link_2_mass" value="1.155" />
+	<xacro:property name="link_3_mass" value="0.934" />
+	<xacro:property name="link_4_mass" value="0.877" />
+	<xacro:property name="link_5_mass" value="0.251" />
+	<!--<xacro:property name="link_0_mass" value="0.845" />
+	<xacro:property name="link_1_mass" value="0.1" />
+	<xacro:property name="link_2_mass" value="0.1" />
+	<xacro:property name="link_3_mass" value="0.1" />
+	<xacro:property name="link_4_mass" value="0.1" />
+	<xacro:property name="link_5_mass" value="0.1" />-->
 	<!-- TODO: add inertia tensor-->
 	<xacro:macro name="default_origin">

File: urdf/youbot_base/base.transmission.xacro (robot description, xacro)
@@ -4,7 +4,7 @@
        xmlns:interface="http://playerstage.sourceforge.net/gazebo/xmlschema/#interface"
        xmlns:xacro="http://ros.org/wiki/xacro">
-	<property name="wheel_mechanical_reduction" value="${624/35 * 80/18}" />
-	<property name="caster_mechanical_reduction" value="${624/35 * 80/18}" />
-	<property name="" value="0.360" />
+	<xacro:property name="wheel_mechanical_reduction" value="${624/35 * 80/18}" />
+	<xacro:property name="caster_mechanical_reduction" value="${624/35 * 80/18}" />
+	<xacro:property name="" value="0.360" />
 	<xacro:macro name="youbot_base_transmission">
 		<!-- front left wheel -->

File: urdf/youbot_gripper/gripper.gazebo.xacro (robot description, xacro)
@@ -1,7 +1,4 @@
 <?xml version="1.0"?>
-<robot xmlns:sensor="http://playerstage.sourceforge.net/gazebo/xmlschema/#sensor"
-       xmlns:controller="http://playerstage.sourceforge.net/gazebo/xmlschema/#controller"
-       xmlns:interface="http://playerstage.sourceforge.net/gazebo/xmlschema/#interface"
-       xmlns:xacro="http://ros.org/wiki/xacro">
+<robot xmlns:xacro="http://ros.org/wiki/xacro">
 	<xacro:macro name="youbot_gripper_gazebo" params="name">
 		<gazebo reference="${name}_palm_link">

File: urdf/youbot_gripper/gripper.transmission.xacro (robot description, xacro)
@@ -1,7 +1,4 @@
 <?xml version="1.0"?>
-<robot xmlns:sensor="http://playerstage.sourceforge.net/gazebo/xmlschema/#sensor"
-       xmlns:controller="http://playerstage.sourceforge.net/gazebo/xmlschema/#controller"
-       xmlns:interface="http://playerstage.sourceforge.net/gazebo/xmlschema/#interface"
-       xmlns:xacro="http://ros.org/wiki/xacro">
+<robot xmlns:xacro="http://ros.org/wiki/xacro">
 	<xacro:macro name="youbot_gripper_transmission" params="name">
 		<transmission name="${name}_finger_l_trans">
@@ -12,5 +9,5 @@
 			</actuator>
 			<joint name="${name}_finger_joint_l">
-				<hardwareInterface>EffortJointInterface</hardwareInterface>
+				<hardwareInterface>hardware_interface/EffortJointInterface</hardwareInterface>
 			</joint>
 		</transmission>
@@ -22,5 +19,5 @@
 			</actuator>
 			<joint name="${name}_finger_joint_r">
-				<hardwareInterface>EffortJointInterface</hardwareInterface>
+				<hardwareInterface>hardware_interface/EffortJointInterface</hardwareInterface>
 			</joint>
 		</transmission>

File: urdf/youbot_gripper/gripper.urdf.xacro (robot description, xacro)
@@ -1,7 +1,4 @@
 <?xml version="1.0"?>
-<robot xmlns:sensor="http://playerstage.sourceforge.net/gazebo/xmlschema/#sensor"
-       xmlns:controller="http://playerstage.sourceforge.net/gazebo/xmlschema/#controller"
-       xmlns:interface="http://playerstage.sourceforge.net/gazebo/xmlschema/#interface"
-       xmlns:xacro="http://ros.org/wiki/xacro">
+<robot xmlns:xacro="http://ros.org/wiki/xacro">
 	<xacro:include filename="$(find youbot_description)/urdf/youbot_gripper/gripper.gazebo.xacro" />
 	<xacro:include filename="$(find youbot_description)/urdf/youbot_gripper/gripper.transmission.xacro" />
@@ -10,5 +7,5 @@
 		<!-- joint between arm_7_link and sdh_palm_link -->
 		<joint name="${name}_palm_joint" type="fixed" >
-			<insert_block name="origin" />
+			<xacro:insert_block name="origin" />
 			<parent link="${parent}" />
 			<child link="${name}_palm_link" />

File: urdf/youbot_gripper/limits.urdf.xacro (robot description, xacro)
@@ -1,9 +1,9 @@
 <?xml version="1.0"?>
-<robot>
+<robot xmlns:xacro="http://www.ros.org/wiki/xacro">
 	<!-- common properties -->
-	<property name="M_PI" value="3.1415926535897931" />
-        <property name="threshold" value="0.001" />
+	<xacro:property name="M_PI" value="3.1415926535897931" />
+        <xacro:property name="threshold" value="0.001" />
 	<!-- fingers limits, values are in meters -->
-	<property name="finger_joint" value="${0.023 / 2.0}" />
-	<property name="finger_joint_soft" value="${(0.023 - threshold) / 2.0}" />
+	<xacro:property name="finger_joint" value="${0.023 / 2.0}" />
+	<xacro:property name="finger_joint_soft" value="${(0.023 - threshold) / 2.0}" />
 </robot>

Commit message: Updated transform to work with normal dh params

File: robots/youbot_arm_only.urdf.xacro (robot description, xacro)
@@ -30,5 +30,5 @@
   </link>
   <xacro:youbot_arm name="$(arg robot_name)" parent="base_link">
-    <origin xyz="0 0 0" rpy="0 0 0" />
+    <origin xyz="-0.024 0 0.030" rpy="0 0 0" />
   </xacro:youbot_arm>
   <xacro:youbot_gripper name="gripper" parent="$(arg robot_name)_link_5">

File: urdf/youbot_arm/arm.urdf.xacro (robot description, xacro)
@@ -211,5 +211,5 @@
           <parent link="${name}_link_5"/>
           <child link="${name}_link_ee"/>
-          <origin xyz="0 0 0.045" rpy="0 0 0"/>
+          <origin xyz="0 0 0.055" rpy="0 0 0"/>
         </joint>
         <link name="${name}_link_ee">
